Commit message: Change frame to base_link for better simulation later

File: src/wheelchair_description/wheelchair/robot.urdf (robot description, URDF)
Before this commit: robot wheelchair, 6 links, 5 joints
Links:
- removed link frame
- added link base_link, mass 109.261; collision mesh filename=package://wheelchair_description/wheelchair/assets/frame.stl; visual mesh filename=package://wheelchair_description/wheelchair/assets/frame.stl
Joints:
- joint back_lw: parent frame -> base_link
- joint back_rw: parent frame -> base_link
- joint chair_joint: parent frame -> base_link
- joint front_lw: parent frame -> base_link
- joint front_rw: parent frame -> base_link

Commit message: Add worlds directory and lidar sensor plugin

File: src/wheelchair_description/wheelchair/robot.urdf (robot description, URDF)
Before this commit: robot wheelchair, 6 links, 5 joints
Links:
- added link lidar_link, mass 0.1; collision cylinder length=0.05 radius=0.03; visual cylinder length=0.05 radius=0.03
Joints:
- added joint lidar_mount: type fixed, parent base_link, child lidar_link, origin xyz=0.3 0 0.025 rpy=0 0 0
